File: diff_drive_pcb/tof.kicad_sch (KiCad schematic)
At the start: 12 parts, among them U4 TOF_front_left, U5 Tof_back_left, U6 Tof_front_right, U7 Tof_back_right, U8 MPU9250

Commit message: Updated Schematic
Parts:
- added D7: headlight, Connector_PinHeader_2.54mm:PinHeader_1x02_P2.54mm_Vertical, symbol Device:LED
- added Q2: IRLZ24, Package_TO_SOT_THT:TO-220-3_Vertical, symbol Transistor_FET:IRLZ24
- added R4: 10k, Resistor_THT:R_Axial_DIN0204_L3.6mm_D1.6mm_P5.08mm_Horizontal, symbol Device:R
- added R5, R6: 100, Resistor_THT:R_Axial_DIN0204_L3.6mm_D1.6mm_P5.08mm_Horizontal, symbol Device:R
Connections:
- net +5V: now also Q2.2 (D), R5.1, R6.1
- net GND: now also D7.1 (K), Q2.3 (S), R4.2
- net HEADLIGHTS: now also Q2.1 (G), R4.1; no longer D6.2 (A)
- new net: D7.2 (A), R6.2
- new net: D6.2 (A), R5.2
- no-connect marks 0 -> 10
Other:
- moved on the sheet: D6

Commit message: Cleaned up PCB and adjusted size
Parts:
- U4, U5, U6, U7: footprint Connector_JST:JST_XH_B6B-XH-AM_1x06_P2.50mm_Vertical -> Connector_JST:JST_XH_B6B-XH-A_1x06_P2.50mm_Vertical
Changed lines of the file:
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@@
 			)
 		)
-		(property "Footprint" "Connector_JST:JST_XH_B6B-XH-AM_1x06_P2.50mm_Vertical"
+		(property "Footprint" "Connector_JST:JST_XH_B6B-XH-A_1x06_P2.50mm_Vertical"
 			(at 41.91 74.93 0)
 			(effects
@@
 			)
 		)
-		(property "Footprint" "Connector_JST:JST_XH_B6B-XH-AM_1x06_P2.50mm_Vertical"
+		(property "Footprint" "Connector_JST:JST_XH_B6B-XH-A_1x06_P2.50mm_Vertical"
 			(at 76.2 39.37 0)
 			(effects
@@
 			)
 		)
-		(property "Footprint" "Connector_JST:JST_XH_B6B-XH-AM_1x06_P2.50mm_Vertical"
+		(property "Footprint" "Connector_JST:JST_XH_B6B-XH-A_1x06_P2.50mm_Vertical"
 			(at 76.2 74.93 0)
 			(effects
@@
 			)
 		)
-		(property "Footprint" "Connector_JST:JST_XH_B6B-XH-AM_1x06_P2.50mm_Vertical"
+		(property "Footprint" "Connector_JST:JST_XH_B6B-XH-A_1x06_P2.50mm_Vertical"
 			(at 41.91 39.37 0)
 			(effects
